Commit message: Рабочий прототип: управление роботом в Gazebo через FMS (интерактивный режим w/a/s/d)

File: robot/amr_hardware/urdf/simple_robot.urdf (robot description, URDF)
Before this commit: robot simple_robot, 3 links, 2 joints
Links:
- added link caster_wheel, mass 0.1; collision sphere radius=0.02; visual sphere radius=0.02
- link left_wheel: geometry collision cylinder length=0.03 radius=0.05; visual cylinder length=0.03 radius=0.05
- link right_wheel: geometry collision cylinder length=0.03 radius=0.05; visual cylinder length=0.03 radius=0.05
Joints:
- added joint base_to_caster: type fixed, parent base_link, child caster_wheel, origin xyz=-0.15 0 -0.05 rpy=0 0 0
- joint base_to_left_wheel: axis 0 0 1 -> 0 1 0; origin xyz=0 0.2 0.05 rpy=1.5708 0 0 -> xyz=0 0.175 -0.05 rpy=0 0 0
- joint base_to_right_wheel: axis 0 0 1 -> 0 1 0; origin xyz=0 -0.2 0.05 rpy=1.5708 0 0 -> xyz=0 -0.175 -0.05 rpy=0 0 0
